File: schematic/Compass.kicad_sch (KiCad schematic)
At the start: 0 parts

Commit message: Create compass schematic
Parts:
- added C10: 0.22uF, symbol Device:C
- added C11: 4.7uF, symbol Device:C
- added C8: 10uF, symbol Device:C
- added C9: 100uF, symbol Device:C
- added R6, R7: 4.7k, symbol Device:R
- added U3: HMC5883L-TR, HMC5883L-TR:XDCR_HMC5883L-TR, symbol HMC5883L-TR:HMC5883L-TR
Connections:
- new net: C11.2, U3.10 (C1)
- new net: C10.1, U3.12 (SETC)
- new net: C10.2, U3.8 (SETP)
- new net +3.3V: C8.1, C9.1, R6.1, R7.1, U3.13 (VDDIO), U3.2 (VDD), U3.4 (S1)
- new net GND: C11.1, C8.2, C9.2, U3.11 (GND), U3.9 (GND)
- new net SCL: R7.2, U3.1 (SCL)
- new net SDA: R6.2, U3.16 (SDA)
- no-connect marks 0 -> 1

Commit message: Assign footprints
Parts:
- C10, C11, C8, C9: footprint (none) -> Capacitor_SMD:C_0603_1608Metric
- R6, R7: footprint (none) -> Resistor_SMD:R_0603_1608Metric
- U3: footprint HMC5883L-TR:XDCR_HMC5883L-TR -> HMC5883L:XDCR_HMC5883L-TR
Changed lines of the file:
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@@
       (effects (font (size 1.27 1.27)))
     )
-    (property "Footprint" "HMC5883L-TR:XDCR_HMC5883L-TR" (at 152.4 101.6 0)
+    (property "Footprint" "HMC5883L:XDCR_HMC5883L-TR" (at 152.4 101.6 0)
       (effects (font (size 1.27 1.27)) (justify bottom) hide)
     )
@@
       (effects (font (size 1.27 1.27)) (justify right))
     )
-    (property "Footprint" "" (at 126.0348 111.76 0)
+    (property "Footprint" "Capacitor_SMD:C_0603_1608Metric" (at 126.0348 111.76 0)
       (effects (font (size 1.27 1.27)) hide)
     )
@@
       (effects (font (size 1.27 1.27)) (justify left))
     )
-    (property "Footprint" "" (at 178.7652 99.06 0)
+    (property "Footprint" "Capacitor_SMD:C_0603_1608Metric" (at 178.7652 99.06 0)
       (effects (font (size 1.27 1.27)) hide)
     )
@@
       (effects (font (size 1.27 1.27)) (justify left))
     )
-    (property "Footprint" "" (at 191.4652 99.06 0)
+    (property "Footprint" "Capacitor_SMD:C_0603_1608Metric" (at 191.4652 99.06 0)
       (effects (font (size 1.27 1.27)) hide)
     )
@@
       (effects (font (size 1.27 1.27)) (justify left))
     )
-    (property "Footprint" "" (at 122.682 80.01 90)
+    (property "Footprint" "Resistor_SMD:R_0603_1608Metric" (at 122.682 80.01 90)
       (effects (font (size 1.27 1.27)) hide)
     )
@@
       (effects (font (size 1.27 1.27)))
     )
-    (property "Footprint" "" (at 132.08 98.0948 0)
+    (property "Footprint" "Capacitor_SMD:C_0603_1608Metric" (at 132.08 98.0948 0)
       (effects (font (size 1.27 1.27)) hide)
     )
@@
       (effects (font (size 1.27 1.27)) (justify left))
     )
-    (property "Footprint" "" (at 132.842 80.01 90)
-      (effects (font (size 1.27 1.27)) hide)
-    )
+    (property "Footprint" "Resistor_SMD:R_0603_1608Metric" (at 132.842 80.01 90)
+      (effects (font (size 1.27 1.27)) hide)
+    )

Commit message: Setup PCB for production
Parts:
- C10: LCSC (none) -> C472764
- C11: LCSC (none) -> C307469
- C8: LCSC (none) -> C19702
- C9: LCSC (none) -> C730416
- R6, R7: LCSC (none) -> C23162
- U3: LCSC (none) -> C976032
Changed lines of the file:
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@@
       (effects (font (size 1.27 1.27)) (justify bottom) hide)
+    )
+    (property "LCSC" "C976032" (at 152.4 101.6 0)
+      (effects (font (size 1.27 1.27)) hide)
     )
     (pin "1")
@@
       (effects (font (size 1.27 1.27)) hide)
     )
+    (property "LCSC" "C307469" (at 127 115.57 0)
+      (effects (font (size 1.27 1.27)) hide)
+    )
     (pin "1")
     (pin "2")
@@
       (effects (font (size 1.27 1.27)) hide)
     )
+    (property "LCSC" "C19702" (at 177.8 95.25 0)
+      (effects (font (size 1.27 1.27)) hide)
+    )
     (pin "1")
     (pin "2")
@@
       (effects (font (size 1.27 1.27)) hide)
     )
+    (property "LCSC" "C730416" (at 190.5 95.25 0)
+      (effects (font (size 1.27 1.27)) hide)
+    )
     (pin "1")
     (pin "2")
@@
       (effects (font (size 1.27 1.27)) hide)
     )
+    (property "LCSC" "C23162" (at 124.46 80.01 0)
+      (effects (font (size 1.27 1.27)) hide)
+    )
     (pin "1")
     (pin "2")
@@
       (effects (font (size 1.27 1.27)) hide)
     )
+    (property "LCSC" "C472764" (at 128.27 99.06 0)
+      (effects (font (size 1.27 1.27)) hide)
+    )
     (pin "1")
     (pin "2")
@@
       (effects (font (size 1.27 1.27)) hide)
     )
+    (property "LCSC" "C23162" (at 134.62 80.01 0)
+      (effects (font (size 1.27 1.27)) hide)
+    )
