File: schematic/ESP32.kicad_sch (KiCad schematic)
At the start: 0 parts

Commit message: Create ESP32 schematic
Parts:
- added C5: 0.1uF, symbol Device:C
- added C6, C7: 10uF, symbol Device:C
- added J2: PROG, symbol Connector:Conn_01x06_Pin
- added Q1, Q2: BC817, Package_TO_SOT_SMD:SOT-23, symbol Transistor_BJT:BC817
- added R3, R4, R5: 10k, symbol Device:R
- added U2: ESP-WROOM-32, ESP-WROOM-32:MODULE_ESP-WROOM-32, symbol ESP-WROOM-32:ESP-WROOM-32
Connections:
- new net: Q2.1 (B), R5.2
- new net: Q2.3 (C), U2.25 (IO0)
- new net: C7.1, Q1.3 (C), R3.2, U2.3 (EN)
- new net: Q1.1 (B), R4.2
- new net +3.3V: C5.1, C6.1, J2.1 (Pin_1), R3.1, U2.2 (3V3)
- new net COMPASS_SCL: U2.36 (IO22)
- new net COMPASS_SDA: U2.33 (IO21)
- new net GND: C5.2, C6.2, C7.2, J2.2 (Pin_2), U2.1 (GND), U2.1.1 (GND), U2.15 (GND), U2.38 (GND)
- new net PROG_DTR: J2.5 (Pin_5), Q2.2 (E), R4.1
- new net PROG_RTS: J2.6 (Pin_6), Q1.2 (E), R5.1
- new net PROG_RX: J2.3 (Pin_3), U2.34 (RXD0)
- new net PROG_TX: J2.4 (Pin_4), U2.35 (TXD0)
- new net SERVO: U2.8 (IO32)
- new net STEPPER_A: U2.37 (IO23)
- new net STEPPER_B: U2.10 (IO25)
- new net STEPPER_C: U2.11 (IO26)
- new net STEPPER_D: U2.12 (IO27)
- no-connect marks 0 -> 22

Commit message: Assign footprints
Parts:
- C5, C6, C7: footprint (none) -> Capacitor_SMD:C_0603_1608Metric
- J2: footprint (none) -> Connector_PinHeader_2.54mm:PinHeader_1x06_P2.54mm_Vertical
- R3, R4, R5: footprint (none) -> Resistor_SMD:R_0603_1608Metric
Changed lines of the file:
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@@
       (effects (font (size 1.27 1.27)))
     )
-    (property "Footprint" "" (at 210.82 93.98 0)
+    (property "Footprint" "Connector_PinHeader_2.54mm:PinHeader_1x06_P2.54mm_Vertical" (at 210.82 93.98 0)
       (effects (font (size 1.27 1.27)) hide)
     )
@@
       (effects (font (size 1.27 1.27)))
     )
-    (property "Footprint" "" (at 69.85 108.458 90)
+    (property "Footprint" "Resistor_SMD:R_0603_1608Metric" (at 69.85 108.458 90)
       (effects (font (size 1.27 1.27)) hide)
     )
@@
       (effects (font (size 1.27 1.27)) (justify left))
     )
-    (property "Footprint" "" (at 97.4852 78.74 0)
+    (property "Footprint" "Capacitor_SMD:C_0603_1608Metric" (at 97.4852 78.74 0)
       (effects (font (size 1.27 1.27)) hide)
     )
@@
       (effects (font (size 1.27 1.27)))
     )
-    (property "Footprint" "" (at 69.85 77.978 90)
+    (property "Footprint" "Resistor_SMD:R_0603_1608Metric" (at 69.85 77.978 90)
       (effects (font (size 1.27 1.27)) hide)
     )
@@
       (effects (font (size 1.27 1.27)) (justify left))
     )
-    (property "Footprint" "" (at 94.742 62.23 90)
+    (property "Footprint" "Resistor_SMD:R_0603_1608Metric" (at 94.742 62.23 90)
       (effects (font (size 1.27 1.27)) hide)
     )
@@
       (effects (font (size 1.27 1.27)) (justify left))
     )
-    (property "Footprint" "" (at 166.0652 73.66 0)
+    (property "Footprint" "Capacitor_SMD:C_0603_1608Metric" (at 166.0652 73.66 0)
       (effects (font (size 1.27 1.27)) hide)
     )
@@
       (effects (font (size 1.27 1.27)) (justify left))
     )
-    (property "Footprint" "" (at 178.7652 73.66 0)
+    (property "Footprint" "Capacitor_SMD:C_0603_1608Metric" (at 178.7652 73.66 0)
       (effects (font (size 1.27 1.27)) hide)
     )

Commit message: Setup PCB for production
Parts:
- C5: LCSC (none) -> C1591
- C6, C7: LCSC (none) -> C19702
- Q1, Q2: LCSC (none) -> C475629
- R3, R4, R5: LCSC (none) -> C25804
- U2: LCSC (none) -> C82899
Changed lines of the file:
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@@
       (effects (font (size 1.27 1.27)) (justify left) hide)
+    )
+    (property "LCSC" "C475629" (at 81.28 106.68 0)
+      (effects (font (size 1.27 1.27)) hide)
     )
     (pin "1")
@@
     )
     (property "Datasheet" "~" (at 210.82 93.98 0)
+      (effects (font (size 1.27 1.27)) hide)
+    )
+    (property "LCSC" "" (at 210.82 93.98 0)
       (effects (font (size 1.27 1.27)) hide)
     )
@@
       (effects (font (size 1.27 1.27)) hide)
     )
+    (property "LCSC" "C25804" (at 69.85 106.68 0)
+      (effects (font (size 1.27 1.27)) hide)
+    )
     (pin "1")
     (pin "2")
@@
       (effects (font (size 1.27 1.27)) hide)
     )
+    (property "LCSC" "C19702" (at 96.52 74.93 0)
+      (effects (font (size 1.27 1.27)) hide)
+    )
     (pin "1")
     (pin "2")
@@
       (effects (font (size 1.27 1.27)) hide)
     )
+    (property "LCSC" "C25804" (at 69.85 76.2 0)
+      (effects (font (size 1.27 1.27)) hide)
+    )
     (pin "1")
     (pin "2")
@@
       (effects (font (size 1.27 1.27)) hide)
     )
+    (property "LCSC" "C25804" (at 96.52 62.23 0)
+      (effects (font (size 1.27 1.27)) hide)
+    )
     (pin "1")
     (pin "2")
@@
       (effects (font (size 1.27 1.27)) hide)
     )
+    (property "LCSC" "C1591" (at 165.1 69.85 0)
+      (effects (font (size 1.27 1.27)) hide)
+    )
     (pin "1")
     (pin "2")
@@
     )
     (property "Datasheet" "~" (at 177.8 69.85 0)
+      (effects (font (size 1.27 1.27)) hide)
+    )
+    (property "LCSC" "C19702" (at 177.8 69.85 0)
       (effects (font (size 1.27 1.27)) hide)
     )
@@
       (effects (font (size 1.27 1.27)) (justify left) hide)
     )
+    (property "LCSC" "C475629" (at 81.28 76.2 0)
+      (effects (font (size 1.27 1.27)) hide)
+    )
     (pin "1")
     (pin "2")
@@
       (effects (font (size 1.27 1.27)) (justify bottom) hide)
     )
-    (pin "1")
+    (property "LCSC" "C82899" (at 139.7 88.9 0)
+      (effects (font (size 1.27 1.27)) hide)
+    )
+    (pin "1")
